File: hardware/pcb/kicad/monitoring-board.kicad_pcb (KiCad board)
At the start: 2 copper layers, 100 x 70 mm, 59 parts, among them IC1 HCPL-7800A-300E, IC2 OP27GSZ, IC3 OP27GSZ, U1 HXS 20-NP/SP30, U2 ESP32-DEVKITC-32E

Commit message: Add project KiCad libraries and publish BOM tables
Parts:
- Alimentacion_Ext_5V1: footprint footprints:Header_TE_640456-2 -> footprints:header-640456-2
- C1: footprint footprints:CapCeramico1000pF_885012207060 -> footprints:capacitor-885012207060
- C10, C11, C3, C4, C6, C8: footprint footprints:CapTantalio0.1uF_TAJS104K020RNJ -> footprints:capacitor-TAJS104K020RNJ
- C12, C14, C5, C7: footprint footprints:CapCeramico200pF_C1206C201F4HACTU -> footprints:capacitor-C1206C201F4HACTU
- C13: footprint footprints:CapCeramico3.3nF_C0805C332F5GECAUTO7210 -> footprints:capacitor-C0805C332F5GECAUTO7210
- C2, C9: footprint footprints:CapElecSMD_KEMET_EXV106M025A9BAA -> footprints:capacitor-EXV106M025A9BAA
- G***: footprint footprints:udc_Logo -> footprints:UDC-logo
- G***: footprint footprints:uaslp_Logo -> footprints:UASLP-logo
- IC1: footprint footprints:SMD_HCPL7800A300E -> footprints:HCPL-7800A-300E
- IC2, IC3: footprint footprints:SMD_OP27GSZ -> footprints:OP27GSZ
- PS_HV1, PS_LV1: footprint footprints:RB-0505D_Convertidor -> footprints:RB-0505D
- R10, R11, R18, R19, R6, R7, R8, R9: footprint footprints:Res1OhmSMD_RCC12061R00FKEA -> footprints:resistor-RCC12061R00FKEA
- R12, R16: footprint footprints:CRGH1206J82K. -> footprints:resistor-CRGH1206J82K
- R13: footprint footprints:CRCW120610K0FKEAC -> footprints:resistor-CRCW120610K0FKEAC
- R14: footprint footprints:Res3.3k_CR0805-FX-3301ELF -> footprints:resistor-CR0805-FX-3301ELF
- R15, R17: footprint footprints:Res100k_CR1206-FX-1003ELF -> footprints:resistor-CR1206-FX-1003ELF
- TP_GND1, TP_GND2, TP_GNDREF1, TP_GNDREF2, TP_GNDREF3, TP_Vin1, TP_Vout1, TP_Vx1, TP_Vy1, TP_sensorCorriente1, TP_sensorVoltaje1: footprint footprints:TestPoint_5001 -> footprints:test-point-5001
- U1: footprint footprints:HXS 20-NP&slash_SP30_LEM -> footprints:HXS20-NP-SP30
- U2: footprint footprints:MODULE_ESP32-DEVKITC-32E -> footprints:ESP32-DEVKITC-32E
