File: hardware/pcb/kicad/monitoring-board.kicad_sch (KiCad schematic)
At the start: 58 parts, among them IC1 HCPL-7800A-300E, IC2 OP27GSZ, IC3 OP27GSZ, J2 USB_B_Micro_2.0, U1 HXS 20-NP/SP30, U2 ESP32-DEVKITC-32E

Commit message: Add project KiCad libraries and publish BOM tables
Parts:
- C1: footprint footprints:CapCeramico1000pF_885012207060 -> footprints:capacitor-885012207060
- C10, C11, C3, C4, C6, C8: footprint footprints:CapTantalio0.1uF_TAJS104K020RNJ -> footprints:capacitor-TAJS104K020RNJ
- C12, C14, C5, C7: footprint footprints:CapCeramico200pF_C1206C201F4HACTU -> footprints:capacitor-C1206C201F4HACTU
- C13: footprint footprints:CapCeramico3.3nF_C0805C332F5GECAUTO7210 -> footprints:capacitor-C0805C332F5GECAUTO7210
- C2, C9: footprint footprints:CapElecSMD_KEMET_EXV106M025A9BAA -> footprints:capacitor-EXV106M025A9BAA
- IC1: footprint footprints:SMD_HCPL7800A300E -> footprints:HCPL-7800A-300E
- IC2, IC3: footprint footprints:SMD_OP27GSZ -> footprints:OP27GSZ
- PS_HV1, PS_LV1: footprint footprints:RB-0505D_Convertidor -> footprints:RB-0505D
- Power_Ext_5V1: footprint footprints:Header_TE_640456-2 -> footprints:header-640456-2
- R10, R11, R18, R19, R6, R7, R8, R9: footprint footprints:Res1OhmSMD_RCC12061R00FKEA -> footprints:resistor-RCC12061R00FKEA
- R12, R16: footprint footprints:CRGH1206J82K. -> footprints:resistor-CRGH1206J82K
- R13: footprint footprints:CRCW120610K0FKEAC -> footprints:resistor-CRCW120610K0FKEAC
- R14: footprint footprints:Res3.3k_CR0805-FX-3301ELF -> footprints:resistor-CR0805-FX-3301ELF
- R15, R17: footprint footprints:Res100k_CR1206-FX-1003ELF -> footprints:resistor-CR1206-FX-1003ELF
- TP_GND1, TP_GND2, TP_GNDREF1, TP_GNDREF2, TP_GNDREF3, TP_Vin1, TP_VoltageSensor, TP_Vout1, TP_Vx1, TP_Vy1, TP_currentSensor: footprint footprints:TestPoint_5001 -> footprints:test-point-5001
- U1: footprint footprints:HXS 20-NP&slash_SP30_LEM -> footprints:HXS20-NP-SP30
- U2: footprint footprints:MODULE_ESP32-DEVKITC-32E -> footprints:ESP32-DEVKITC-32E
Changed lines of the file:
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@@
 			)
 		)
-		(property "Footprint" "footprints:Res1OhmSMD_RCC12061R00FKEA"
+		(property "Footprint" "footprints:resistor-RCC12061R00FKEA"
 			(at 154.94 50.038 90)
 			(effects
@@
 			)
 		)
-		(property "Footprint" "footprints:CapTantalio0.1uF_TAJS104K020RNJ"
+		(property "Footprint" "footprints:capacitor-TAJS104K020RNJ"
 			(at 177.8 69.85 0)
 			(effects
@@
 			)
 		)
-		(property "Footprint" "footprints:SMD_HCPL7800A300E"
+		(property "Footprint" "footprints:HCPL-7800A-300E"
 			(at 137.16 140.64 0)
 			(effects
@@
 			)
 		)
-		(property "Footprint" "footprints:CapCeramico200pF_C1206C201F4HACTU"
+		(property "Footprint" "footprints:capacitor-C1206C201F4HACTU"
 			(at 199.39 25.7048 0)
 			(effects
@@
 			)
 		)
-		(property "Footprint" "footprints:SMD_OP27GSZ"
+		(property "Footprint" "footprints:OP27GSZ"
 			(at 209.55 135.56 0)
 			(effects
@@
 			)
 		)
-		(property "Footprint" "footprints:RB-0505D_Convertidor"
+		(property "Footprint" "footprints:RB-0505D"
 			(at 68.58 248.59 0)
 			(effects
@@
 			)
 		)
-		(property "Footprint" "footprints:CapElecSMD_KEMET_EXV106M025A9BAA"
+		(property "Footprint" "footprints:capacitor-EXV106M025A9BAA"
 			(at 92.71 50.8 0)
 			(effects
@@
 			)
 		)
-		(property "Footprint" "footprints:TestPoint_5001"
+		(property "Footprint" "footprints:test-point-5001"
 			(at 312.09 29.21 0)
 			(effects
@@
 			)
 		)
-		(property "Footprint" "footprints:Res1OhmSMD_RCC12061R00FKEA"
+		(property "Footprint" "footprints:resistor-RCC12061R00FKEA"
 			(at 87.63 47.498 90)
 			(effects
@@
 			)
 		)
-		(property "Footprint" "footprints:CapCeramico200pF_C1206C201F4HACTU"
+		(property "Footprint" "footprints:capacitor-C1206C201F4HACTU"
 			(at 164.7952 62.23 0)
 			(effects
@@
 			)
 		)
-		(property "Footprint" "footprints:Res100k_CR1206-FX-1003ELF"
+		(property "Footprint" "footprints:resistor-CR1206-FX-1003ELF"
 			(at 223.52 69.088 90)
 			(effects
@@
 			)
 		)
-		(property "Footprint" "footprints:Header_TE_640456-2"
+		(property "Footprint" "footprints:header-640456-2"
 			(at 40.64 144.78 0)
 			(effects
@@
 			)
 		)
-		(property "Footprint" "footprints:CapTantalio0.1uF_TAJS104K020RNJ"
+		(property "Footprint" "footprints:capacitor-TAJS104K020RNJ"
 			(at 137.16 66.04 0)
 			(effects
@@
 			)
 		)
-		(property "Footprint" "footprints:CapTantalio0.1uF_TAJS104K020RNJ"
+		(property "Footprint" "footprints:capacitor-TAJS104K020RNJ"
 			(at 251.46 80.01 0)
 			(effects
@@
 			)
 		)
-		(property "Footprint" "footprints:TestPoint_5001"
+		(property "Footprint" "footprints:test-point-5001"
 			(at -40.31 45.72 0)
 			(effects
@@
 			)
 		)
-		(property "Footprint" "footprints:CapElecSMD_KEMET_EXV106M025A9BAA"
+		(property "Footprint" "footprints:capacitor-EXV106M025A9BAA"
 			(at 208.28 72.39 0)
 			(effects
@@
 			)
 		)
-		(property "Footprint" "footprints:Res1OhmSMD_RCC12061R00FKEA"
+		(property "Footprint" "footprints:resistor-RCC12061R00FKEA"
 			(at 140.97 108.458 90)
 			(effects
@@
 			)
 		)
-		(property "Footprint" "footprints:TestPoint_5001"
+		(property "Footprint" "footprints:test-point-5001"
 			(at 181.94 86.36 0)
 			(effects
@@
 			)
 		)
-		(property "Footprint" "footprints:HXS 20-NP&slash_SP30_LEM"
+		(property "Footprint" "footprints:HXS20-NP-SP30"
 			(at 29.21 109.22 0)
 			(effects
@@
 			)
 		)
-		(property "Footprint" "footprints:Res3.3k_CR0805-FX-3301ELF"
+		(property "Footprint" "footprints:resistor-CR0805-FX-3301ELF"
 			(at 212.852 72.39 90)
 			(effects
@@
 			)
 		)
-		(property "Footprint" "footprints:TestPoint_5001"
+		(property "Footprint" "footprints:test-point-5001"
 			(at 48.59 68.58 0)
 			(effects
@@
 			)
 		)
-		(property "Footprint" "footprints:TestPoint_5001"
+		(property "Footprint" "footprints:test-point-5001"
 			(at 153.34 68.58 0)
 			(effects
@@
 			)
 		)
-		(property "Footprint" "footprints:SMD_OP27GSZ"
+		(property "Footprint" "footprints:OP27GSZ"
 			(at 275.59 133.02 0)
 			(effects
@@
 			)
 		)
-		(property "Footprint" "footprints:MODULE_ESP32-DEVKITC-32E"
+		(property "Footprint" "footprints:ESP32-DEVKITC-32E"
 			(at 129.54 170.18 0)
 			(effects
@@
 			)
 		)
-		(property "Footprint" "footprints:TestPoint_5001"
+		(property "Footprint" "footprints:test-point-5001"
 			(at 128.27 4.14 0)
 			(effects
@@
 			)
 		)
-		(property "Footprint" "footprints:CapCeramico3.3nF_C0805C332F5GECAUTO7210"
+		(property "Footprint" "footprints:capacitor-C0805C332F5GECAUTO7210"
 			(at 120.3452 111.76 0)
 			(effects
@@
 			)
 		)
-		(property "Footprint" "footprints:Res1OhmSMD_RCC12061R00FKEA"
+		(property "Footprint" "footprints:resistor-RCC12061R00FKEA"
 			(at 152.4 108.458 90)
 			(effects
@@
 			)
 		)
-		(property "Footprint" "footprints:RB-0505D_Convertidor"
+		(property "Footprint" "footprints:RB-0505D"
 			(at 68.58 271.45 0)
 			(effects
@@
 			)
 		)
-		(property "Footprint" "footprints:CapTantalio0.1uF_TAJS104K020RNJ"
+		(property "Footprint" "footprints:capacitor-TAJS104K020RNJ"
 			(at 182.88 69.85 0)
 			(effects
@@
 			)
 		)
-		(property "Footprint" "footprints:CRGH1206J82K."
+		(property "Footprint" "footprints:resistor-CRGH1206J82K"
 			(at 228.6 37.338 90)
 			(effects
@@
 			)
 		)
-		(property "Footprint" "footprints:TestPoint_5001"
+		(property "Footprint" "footprints:test-point-5001"
 			(at 10.49 74.93 0)
 			(effects
@@
 			)
 		)
-		(property "Footprint" "footprints:Res1OhmSMD_RCC12061R00FKEA"
+		(property "Footprint" "footprints:resistor-RCC12061R00FKEA"
 			(at 195.58 22.098 90)
 			(effects
@@
 			)
 		)
-		(property "Footprint" "footprints:TestPoint_5001"
+		(property "Footprint" "footprints:test-point-5001"
 			(at 157.48 167.31 0)
 			(effects
@@
 			)
 		)
-		(property "Footprint" "footprints:Res1OhmSMD_RCC12061R00FKEA"
+		(property "Footprint" "footprints:resistor-RCC12061R00FKEA"
 			(at 159.258 58.42 90)
 			(effects
@@
 			)
 		)
-		(property "Footprint" "footprints:TestPoint_5001"
+		(property "Footprint" "footprints:test-point-5001"
 			(at 14.3 74.93 0)
 			(effects
@@
 			)
 		)
-		(property "Footprint" "footprints:CRCW120610K0FKEAC"
+		(property "Footprint" "footprints:resistor-CRCW120610K0FKEAC"
 			(at 212.852 60.96 90)
 			(effects
@@
 			)
 		)
-		(property "Footprint" "footprints:Res100k_CR1206-FX-1003ELF"
+		(property "Footprint" "footprints:resistor-CR1206-FX-1003ELF"
 			(at 260.35 22.098 90)
 			(effects
@@
 			)
 		)
-		(property "Footprint" "footprints:CRGH1206J82K."
+		(property "Footprint" "footprints:resistor-CRGH1206J82K"
 			(at 223.52 47.498 90)
 			(effects
@@
 			)
 		)
-		(property "Footprint" "footprints:Res1OhmSMD_RCC12061R00FKEA"
+		(property "Footprint" "footprints:resistor-RCC12061R00FKEA"
 			(at 78.74 50.038 90)
 			(effects
@@
 			)
 		)
-		(property "Footprint" "footprints:CapCeramico200pF_C1206C201F4HACTU"
+		(property "Footprint" "footprints:capacitor-C1206C201F4HACTU"
 			(at 129.2352 116.84 0)
 			(effects
@@
 			)
 		)
-		(property "Footprint" "footprints:CapTantalio0.1uF_TAJS104K020RNJ"
+		(property "Footprint" "footprints:capacitor-TAJS104K020RNJ"
 			(at 97.79 50.8 0)
 			(effects
@@
 			)
 		)
-		(property "Footprint" "footprints:CapCeramico1000pF_885012207060"
+		(property "Footprint" "footprints:capacitor-885012207060"
 			(at 84.7852 62.23 0)
 			(effects
@@
 			)
 		)
-		(property "Footprint" "footprints:TestPoint_5001"
+		(property "Footprint" "footprints:test-point-5001"
 			(at 157.48 163.5 0)
 			(effects
@@
 			)
 		)
-		(property "Footprint" "footprints:CapTantalio0.1uF_TAJS104K020RNJ"
+		(property "Footprint" "footprints:capacitor-TAJS104K020RNJ"
 			(at 243.84 80.01 0)
 			(effects
@@
 			)
 		)
-		(property "Footprint" "footprints:CapCeramico200pF_C1206C201F4HACTU"
+		(property "Footprint" "footprints:capacitor-C1206C201F4HACTU"
 			(at 111.4552 109.22 0)
 			(effects
@@
 			)
 		)
-		(property "Footprint" "footprints:Res1OhmSMD_RCC12061R00FKEA"
+		(property "Footprint" "footprints:resistor-RCC12061R00FKEA"
 			(at 158.75 44.958 90)
 			(effects
@@
 			)
 		)
-		(property "Footprint" "footprints:TestPoint_5001"
+		(property "Footprint" "footprints:test-point-5001"
 			(at 157.48 171.12 0)
 			(effects
